Commit message: Added base link code & features.

File: urdf/Robot.urdf (robot description, URDF)
Before this commit: robot autonomous_sphere_collector, 5 links, 4 joints
Links:
- removed link caster_wheel
- removed link left_wheel
- removed link lidar
- removed link right_wheel
Joints:
- removed joint base_caster_wheel
- removed joint base_left_wheel
- removed joint base_lidar_joint
- removed joint base_right_wheel

Commit message: Added Lidar link code & features

File: urdf/Robot.urdf (robot description, URDF)
Before this commit: robot autonomous_sphere_collector, 1 links, 0 joints
Links:
- added link lidar; visual cylinder length=0.05 radius=0.1

Commit message: Added left,right wheel link,Code,features

File: urdf/Robot.urdf (robot description, URDF)
Before this commit: robot autonomous_sphere_collector, 2 links, 0 joints
Links:
- added link left_wheel; visual cylinder length=0.05 radius=0.1
- added link right_wheel; visual cylinder length=0.05 radius=0.1

Commit message: Added caster wheel link,code,feature

File: urdf/Robot.urdf (robot description, URDF)
Before this commit: robot autonomous_sphere_collector, 4 links, 0 joints
Links:
- added link caster_wheel; visual sphere radius=0.05

Commit message: Attach lidar to base_link via base_lidar_joint.

File: urdf/Robot.urdf (robot description, URDF)
Before this commit: robot autonomous_sphere_collector, 5 links, 0 joints
Joints:
- added joint base_lidar_joint: type fixed, parent base_link, child lidar, origin xyz=0 0 0.225 rpy=0 0 0

Commit message: Defined both wheels joint to base link.

File: urdf/Robot.urdf (robot description, URDF)
Before this commit: robot autonomous_sphere_collector, 5 links, 1 joints
Joints:
- added joint base_left_wheel: type continuous, parent base_link, child left_wheel, origin xyz=-0.15 0.225 0 rpy=0 0 0, axis 0 1 0
- added joint base_right_wheel: type continuous, parent base_link, child right_wheel, origin xyz=-0.15 -0.225 0 rpy=0 0 0, axis 0 1 0

Commit message: Attached caster wheel joint to base link.

File: urdf/Robot.urdf (robot description, URDF)
Before this commit: robot autonomous_sphere_collector, 5 links, 3 joints
Joints:
- added joint base_caster_wheel: type continuous, parent base_link, child caster_wheel, origin xyz=0.2 0 -0.05 rpy=0 0 0, axis 1 1 1

Commit message: Attemp to make a pushing mechanism

File: urdf/Robot.urdf (robot description, URDF)
Before this commit: robot autonomous_sphere_collector, 5 links, 4 joints
Links:
- added link base_footprint
- added link push_plate; visual box size=0.3 0.5 0.01
Joints:
- added joint base_push_plate: type revolute, parent base_link, child push_plate, origin xyz=0.3 0 0.1 rpy=0 0 0, axis 0 1 0, limit lower=-1.57 upper=1.57 effort=10 velocity=1.0
- added joint footprint_base_joint: type fixed, parent base_footprint, child base_link, origin xyz=0 0 0.1 rpy=0 0 0
- joint base_caster_wheel: axis 1 1 1 -> 0 1 0

Commit message: Fixed wheel offset in 'z' and caster type to fixed.

File: urdf/Robot.urdf (robot description, URDF)
Before this commit: robot autonomous_sphere_collector, 7 links, 6 joints
Joints:
- joint base_caster_wheel: type continuous -> fixed
- joint base_left_wheel: origin xyz=-0.15 0.225 0 rpy=0 0 0 -> xyz=-0.15 0.225 0.1 rpy=0 0 0
- joint base_right_wheel: origin xyz=-0.15 -0.225 0 rpy=0 0 0 -> xyz=-0.15 -0.225 0.1 rpy=0 0 0

Commit message: Fixing the gripping mechanism.

File: urdf/Robot.urdf (robot description, URDF)
Before this commit: robot autonomous_sphere_collector, 7 links, 6 joints
Links:
- removed link push_plate
- added link scoop_center; visual box size=0.40 0.04 0.14
- added link scoop_left_wing; visual box size=0.25 0.04 0.14
- added link scoop_right_wing; visual box size=0.25 0.04 0.14
Joints:
- removed joint base_push_plate
- added joint base_bulldozer_scoop: type revolute, parent base_link, child bulldozer_scoop, origin xyz=0.35 0 0.075 rpy=0.3 0 0, axis 0 1 0, limit lower=-1.57 upper=1.57 effort=10 velocity=1.0
- joint base_left_wheel: origin xyz=-0.15 0.225 0.1 rpy=0 0 0 -> xyz=-0.15 0.225 0 rpy=0 0 0
- joint base_right_wheel: origin xyz=-0.15 -0.225 0.1 rpy=0 0 0 -> xyz=-0.15 -0.225 0 rpy=0 0 0

Commit message: Fixinf gripping mechanism

File: urdf/Robot.urdf (robot description, URDF)
Before this commit: robot autonomous_sphere_collector, 9 links, 6 joints
Links:
- removed link scoop_center
- link scoop_left_wing: geometry visual box size=0.1 0.04 0.14
- link scoop_right_wing: geometry visual box size=0.1 0.04 0.14
Joints:
- removed joint base_bulldozer_scoop
- added joint scoop_left_wing_joint: type fixed, parent base_link, child scoop_left_wing, origin xyz=0.30 0.18 0.08 rpy=0.25 0 0.0
- added joint scoop_right_wing_joint: type fixed, parent base_link, child scoop_right_wing, origin xyz=0.30 -0.18 0.08 rpy=0.25 0 0

Commit message: Fixinf gripper mechanism

File: urdf/Robot.urdf (robot description, URDF)
Before this commit: robot autonomous_sphere_collector, 8 links, 7 joints
Links:
- link scoop_left_wing: geometry visual box size=0.1 0.04 0.1
- link scoop_right_wing: geometry visual box size=0.1 0.04 0.1
Joints:
- joint base_caster_wheel: axis 0 1 0 -> (none)
- joint scoop_left_wing_joint: axis (none) -> 0 1 0; limit (none) -> lower=-1.57 upper=1.57 effort=10.0 velocity=1.0; origin xyz=0.30 0.18 0.08 rpy=0.25 0 0.0 -> xyz=0.30 0.18 0.08 rpy=0 0 0.0; type fixed -> revolute
- joint scoop_right_wing_joint: axis (none) -> 0 1 0; limit (none) -> lower=-1.57 upper=1.57 effort=10.0 velocity=1.0; origin xyz=0.30 -0.18 0.08 rpy=0.25 0 0 -> xyz=0.30 -0.18 0.08 rpy=0 0 0; type fixed -> revolute

Commit message: Fixing bucket mechanism.

File: urdf/Robot.urdf (robot description, URDF)
Before this commit: robot autonomous_sphere_collector, 8 links, 7 joints
Links:
- added link bucket; visual box size=0.1 0.2 0.15
Joints:
- added joint left_bucket_joint: type fixed, parent scoop_left_wing, child bucket, origin xyz=0.05 -0.1 0.0 rpy=0 0 0
- added joint right_bucket_joint: type fixed, parent scoop_right_wing, child bucket, origin xyz=0.2 0.1 0.1 rpy=0 0 0

Commit message: Finalizing bucket mechanism

File: urdf/Robot.urdf (robot description, URDF)
Before this commit: robot autonomous_sphere_collector, 9 links, 9 joints
Links:
- removed link bucket
- added link bucket_back_wall; visual box size=0.01 0.3 0.15
- added link bucket_bottom; visual box size=0.1 0.3 0.01
- added link bucket_left_wall; visual box size=0.1 0.01 0.15
Joints:
- removed joint left_bucket_joint
- removed joint right_bucket_joint
- added joint bucket_back_wall_joint: type fixed, parent base_link, child bucket_back_wall, origin xyz=0.325 0 0.08 rpy=0 0 0
- added joint bucket_bottom_joint: type fixed, parent base_link, child bucket_bottom, origin xyz=0.38 0 0.01 rpy=0 0 0
- added joint bucket_left_wall_joint: type fixed, parent base_link, child bucket_left_wall, origin xyz=0.38 0.15 0.08 rpy=0 0 0

Commit message: Defined bucket as gripping mechanism

File: urdf/Robot.urdf (robot description, URDF)
Before this commit: robot autonomous_sphere_collector, 11 links, 10 joints
Links:
- added link bucket_front_lip; visual box size=0.02 0.3 0.005
- added link bucket_right_wall; visual box size=0.1 0.01 0.15
- link scoop_left_wing: geometry visual box size=0.1 0.055 0.05
- link scoop_right_wing: geometry visual box size=0.1 0.055 0.05
Joints:
- added joint bucket_front_lip_joint: type fixed, parent bucket_bottom, child bucket_front_lip, origin xyz=0.059 0.0 0 rpy=0 0.28 0
- added joint bucket_right_wall_joint: type fixed, parent base_link, child bucket_right_wall, origin xyz=0.38 -0.15 0.08 rpy=0 0 0

Commit message: Gripping mechanism completed

File: urdf/Robot.urdf (robot description, URDF)
Before this commit: robot autonomous_sphere_collector, 13 links, 12 joints
Links:
- added link bucket
- link bucket_left_wall: geometry visual box size=0.1 0.006 0.15
- link bucket_right_wall: geometry visual box size=0.1 0.006 0.15
- link scoop_left_wing: geometry visual box size=0.1 0.040 0.05
- link scoop_right_wing: geometry visual box size=0.1 0.040 0.05
Joints:
- added joint bucket_revolute_joint: type fixed, parent scoop_left_wing, child bucket, origin xyz=-0.3 -0.18 -0.015 rpy=0 0 0.0
- joint bucket_back_wall_joint: parent base_link -> bucket
- joint bucket_bottom_joint: parent base_link -> bucket
- joint bucket_left_wall_joint: parent base_link -> bucket
- joint bucket_right_wall_joint: parent base_link -> bucket
- joint scoop_left_wing_joint: origin xyz=0.30 0.18 0.08 rpy=0 0 0.0 -> xyz=0.30 0.18 0.05 rpy=0 0 0
- joint scoop_right_wing_joint: origin xyz=0.30 -0.18 0.08 rpy=0 0 0 -> xyz=0.30 -0.18 0.05 rpy=0 0 0

Commit message: Fixed robot submerging issue

File: urdf/Robot.urdf (robot description, URDF)
Before this commit: robot autonomous_sphere_collector, 14 links, 13 joints
Joints:
- joint base_caster_wheel: origin xyz=0.2 0 -0.05 rpy=0 0 0 -> xyz=0.2 0 -0.07 rpy=0 0 0
- joint base_left_wheel: origin xyz=-0.15 0.225 0 rpy=0 0 0 -> xyz=-0.15 0.225 -0.02 rpy=0 0 0
- joint base_right_wheel: origin xyz=-0.15 -0.225 0 rpy=0 0 0 -> xyz=-0.15 -0.225 -0.02 rpy=0 0 0
- joint footprint_base_joint: origin xyz=0 0 0.1 rpy=0 0 0 -> xyz=0 0 0.12 rpy=0 0 0

Commit message: Defined collison to the robot.

File: urdf/Robot.urdf (robot description, URDF)
Before this commit: robot autonomous_sphere_collector, 14 links, 13 joints
Links:
- link base_link: geometry collision box size=0.6 0.4 0.2; visual box size=0.6 0.4 0.2
- link bucket_back_wall: geometry collision box size=0.01 0.3 0.15; visual box size=0.01 0.3 0.15
- link bucket_bottom: geometry collision box size=0.1 0.3 0.01; visual box size=0.1 0.3 0.01
- link bucket_front_lip: geometry collision box size=0.02 0.3 0.005; visual box size=0.02 0.3 0.005
- link bucket_left_wall: geometry collision box size=0.1 0.006 0.15; visual box size=0.1 0.006 0.15
- link bucket_right_wall: geometry collision box size=0.1 0.006 0.15; visual box size=0.1 0.006 0.15
- link caster_wheel: geometry collision sphere radius=0.05; visual sphere radius=0.05
- link left_wheel: geometry collision cylinder length=0.05 radius=0.1; visual cylinder length=0.05 radius=0.1
- link lidar: geometry collision cylinder length=0.05 radius=0.1; visual cylinder length=0.05 radius=0.1
- link right_wheel: geometry collision cylinder length=0.05 radius=0.1; visual cylinder length=0.05 radius=0.1
- link scoop_left_wing: geometry collision box size=0.1 0.040 0.05; visual box size=0.1 0.040 0.05
- link scoop_right_wing: geometry collision box size=0.1 0.040 0.05; visual box size=0.1 0.040 0.05

Commit message: Defined mass and inertia for physics in gazebo

File: urdf/Robot.urdf (robot description, URDF)
Before this commit: robot autonomous_sphere_collector, 14 links, 13 joints
Links:
- link base_link: mass None -> 10.0
- link bucket_back_wall: mass None -> 0.5
- link bucket_bottom: mass None -> 0.3
- link bucket_front_lip: mass None -> 0.1
- link bucket_left_wall: mass None -> 0.2
- link bucket_right_wall: mass None -> 0.2
- link caster_wheel: mass None -> 0.5
- link left_wheel: mass None -> 1.0
- link right_wheel: mass None -> 1.0
- link scoop_left_wing: mass None -> 0.5
- link scoop_right_wing: mass None -> 0.5

Commit message: Defined IMU ink and joint.

File: urdf/Robot.urdf (robot description, URDF)
Before this commit: robot autonomous_sphere_collector, 15 links, 14 joints
Links:
- added link imu_link, mass 0.05; collision box size=0.08 0.04 0.01; visual box size=0.08 0.04 0.01
Joints:
- added joint imu_joint: type fixed, parent base_link, child imu_link, origin xyz=0.28 0.0 0.220 rpy=0 0 0

Commit message: Fixed IMU origin and dimensions.

File: urdf/Robot.urdf (robot description, URDF)
Before this commit: robot autonomous_sphere_collector, 16 links, 15 joints
Links:
- link imu_link: geometry collision box size=0.04 0.08 0.01; visual box size=0.025 0.08 0.01
Joints:
- joint imu_joint: origin xyz=0.28 0.0 0.220 rpy=0 0 0 -> xyz=0.12 0.0 0.201 rpy=0 0 0

Commit message: Modularized urdf into xacro using macro

File: urdf/Robot.urdf (robot description, URDF)
Before this commit: robot autonomous_sphere_collector, 16 links, 15 joints
Links:
- removed link bucket_back_wall
- removed link bucket_bottom
- removed link bucket_front_lip
- removed link bucket_left_wall
- removed link bucket_right_wall
- removed link camera_link
- removed link caster_wheel
- removed link imu_link
- removed link left_wheel
- removed link lidar
- removed link right_wheel
- removed link scoop_left_wing
- removed link scoop_right_wing
- link base_link: mass 10.0 -> ${base_mass}; geometry collision box size=${base_length} ${base_width} ${base_height}; visual box size=${base_length} ${base_width} ${base_height}
Joints:
- removed joint base_caster_wheel
- removed joint base_left_wheel
- removed joint base_lidar_joint
- removed joint base_right_wheel
- removed joint bucket_back_wall_joint
- removed joint bucket_bottom_joint
- removed joint bucket_front_lip_joint
- removed joint bucket_left_wall_joint
- removed joint bucket_revolute_joint
- removed joint bucket_right_wall_joint
- removed joint camera_joint
- removed joint footprint_base_joint
- removed joint imu_joint
- removed joint scoop_left_wing_joint
- removed joint scoop_right_wing_joint

Commit message: Fixed urdf origin errors trying to convert in xacro

File: urdf/Robot.urdf (robot description, URDF)
Before this commit: robot autonomous_sphere_collector, 3 links, 0 joints
Links:
- added link bucket_back_wall, mass 0.5; collision box size=0.01 0.3 0.15; visual box size=0.01 0.3 0.15
- added link bucket_bottom, mass 0.3; collision box size=0.1 0.3 0.01; visual box size=0.1 0.3 0.01
- added link bucket_front_lip, mass 0.1; collision box size=0.02 0.3 0.005; visual box size=0.02 0.3 0.005
- added link bucket_left_wall, mass 0.2; collision box size=0.1 0.006 0.15; visual box size=0.1 0.006 0.15
- added link bucket_right_wall, mass 0.2; collision box size=0.1 0.006 0.15; visual box size=0.1 0.006 0.15
- added link camera_link, mass 0.1; collision box size=0.05 0.05 0.05; visual box size=0.02 0.07 0.02
- added link caster_wheel, mass 0.5; collision sphere radius=0.05; visual sphere radius=0.05
- added link imu_link, mass 0.05; collision box size=0.04 0.08 0.01; visual box size=0.025 0.08 0.01
- added link left_wheel, mass 1.0; collision cylinder length=0.05 radius=0.1; visual cylinder length=0.05 radius=0.1
- added link lidar; collision cylinder length=0.05 radius=0.1; visual cylinder length=0.05 radius=0.1
- added link right_wheel, mass 1.0; collision cylinder length=0.05 radius=0.1; visual cylinder length=0.05 radius=0.1
- added link scoop_left_wing, mass 0.5; collision box size=0.1 0.040 0.05; visual box size=0.1 0.040 0.05
- added link scoop_right_wing, mass 0.5; collision box size=0.1 0.040 0.05; visual box size=0.1 0.040 0.05
- link base_link: mass ${base_mass} -> 10.0; geometry collision box size=0.6 0.4 0.2; visual box size=0.6 0.4 0.2
Joints:
- added joint base_caster_wheel: type fixed, parent base_link, child caster_wheel, origin xyz=0.2 0 -0.07 rpy=0 0 0
- added joint base_left_wheel: type continuous, parent base_link, child left_wheel, origin xyz=-0.15 0.225 -0.02 rpy=0 0 0, axis 0 1 0
- added joint base_lidar_joint: type fixed, parent base_link, child lidar, origin xyz=0 0 0.225 rpy=0 0 0
- added joint base_right_wheel: type continuous, parent base_link, child right_wheel, origin xyz=-0.15 -0.225 -0.02 rpy=0 0 0, axis 0 1 0
- added joint bucket_back_wall_joint: type fixed, parent bucket, child bucket_back_wall, origin xyz=0.325 0 0.08 rpy=0 0 0
- added joint bucket_bottom_joint: type fixed, parent bucket, child bucket_bottom, origin xyz=0.38 0 0.01 rpy=0 0 0
- added joint bucket_front_lip_joint: type fixed, parent bucket_bottom, child bucket_front_lip, origin xyz=0.059 0.0 0 rpy=0 0.28 0
- added joint bucket_left_wall_joint: type fixed, parent bucket, child bucket_left_wall, origin xyz=0.38 0.15 0.08 rpy=0 0 0
- added joint bucket_revolute_joint: type fixed, parent scoop_left_wing, child bucket, origin xyz=-0.3 -0.18 -0.015 rpy=0 0 0.0
- added joint bucket_right_wall_joint: type fixed, parent bucket, child bucket_right_wall, origin xyz=0.38 -0.15 0.08 rpy=0 0 0
- added joint camera_joint: type fixed, parent base_link, child camera_link, origin xyz=0.30 0.0 0.215 rpy=0 0.20 0
- added joint footprint_base_joint: type fixed, parent base_footprint, child base_link, origin xyz=0 0 0.12 rpy=0 0 0
- added joint imu_joint: type fixed, parent base_link, child imu_link, origin xyz=0.12 0.0 0.201 rpy=0 0 0
- added joint scoop_left_wing_joint: type revolute, parent base_link, child scoop_left_wing, origin xyz=0.30 0.18 0.05 rpy=0 0 0, axis 0 1 0, limit lower=-1.57 upper=1.57 effort=10.0 velocity=1.0
- added joint scoop_right_wing_joint: type revolute, parent base_link, child scoop_right_wing, origin xyz=0.30 -0.18 0.05 rpy=0 0 0, axis 0 1 0, limit lower=-1.57 upper=1.57 effort=10.0 velocity=1.0
