Commit message: Fixed modularity rvixz launch renamed.created xacro and urdf.

File: urdf/Robot.xacro (robot description, xacro)
@@ -1,107 +1,465 @@
 <?xml version="1.0"?>
 <robot xmlns:xacro="http://www.ros.org/wiki/xacro" name="autonomous_sphere_collector">
-  <!-- ==================== PROPERTIES ==================== -->
-  <xacro:property name="base_length" value="0.6"/>
-  <xacro:property name="base_width"  value="0.4"/>
-  <xacro:property name="base_height" value="0.2"/>
-  <xacro:property name="base_mass"   value="10.0"/>
-  <!-- ==================== MATERIALS MACRO ==================== -->
-  <xacro:macro name="define_materials">
-    <material name="grey"><color rgba="0.7 0.7 0.7 1"/></material>
-    <material name="green"><color rgba="0 0.6 0 1"/></material>
-    <material name="white"><color rgba="1 1 1 1"/></material>
-  </xacro:macro>
-  <!-- ==================== LINK MACROS ==================== -->
-  <xacro:macro name="sensor_link" params="name geometry size_x size_y size_z radius length mass material">
-    <link name="${name}">
-      <visual>
-        <geometry>
-          <xacro:if value="${geometry == 'box'}"><box size="${size_x} ${size_y} ${size_z}"/></xacro:if>
-          <xacro:if value="${geometry == 'cylinder'}"><cylinder radius="${radius}" length="${length}"/></xacro:if>
-        </geometry>
-        <origin xyz="0 0 0" rpy="0 0 0"/>
-        <material name="${material}"/>
-      </visual>
-      <collision>
-        <geometry>
-          <xacro:if value="${geometry == 'box'}"><box size="${size_x} ${size_y} ${size_z}"/></xacro:if>
-          <xacro:if value="${geometry == 'cylinder'}"><cylinder radius="${radius}" length="${length}"/></xacro:if>
-        </geometry>
-        <origin xyz="0 0 0" rpy="0 0 0"/>
-      </collision>
-      <inertial>
-        <mass value="${mass}"/>
-        <origin xyz="0 0 0" rpy="0 0 0"/>
-        <inertia ixx="0.0001" iyy="0.0001" izz="0.0001"/>
-      </inertial>
-    </link>
-  </xacro:macro>
-  <xacro:macro name="wheel_link" params="name radius length mass material rpy">
-    <link name="${name}">
-      <visual><geometry><cylinder radius="${radius}" length="${length}"/></geometry><origin xyz="0 0 0" rpy="${rpy}"/><material name="${material}"/></visual>
-      <collision><geometry><cylinder radius="${radius}" length="${length}"/></geometry><origin xyz="0 0 0" rpy="${rpy}"/></collision>
-      <inertial><mass value="${mass}"/><origin xyz="0 0 0" rpy="${rpy}"/><inertia ixx="0.00375" iyy="0.00375" izz="0.005"/></inertial>
-    </link>
-  </xacro:macro>
-  <xacro:macro name="caster_link" params="name radius mass material">
-    <link name="${name}">
-      <visual><geometry><sphere radius="${radius}"/></geometry><origin xyz="0 0 0" rpy="0 0 0"/><material name="${material}"/></visual>
-      <collision><geometry><sphere radius="${radius}"/></geometry><origin xyz="0 0 0" rpy="0 0 0"/></collision>
-      <inertial><mass value="${mass}"/><origin xyz="0 0 0" rpy="0 0 0"/><inertia ixx="0.001" iyy="0.001" izz="0.001"/></inertial>
-    </link>
-  </xacro:macro>
-  <xacro:macro name="wing_link" params="name size_x size_y size_z mass material">
-    <link name="${name}">
-      <visual><geometry><box size="${size_x} ${size_y} ${size_z}"/></geometry><origin xyz="0 0 0" rpy="0 0 0"/><material name="${material}"/></visual>
-      <collision><geometry><box size="${size_x} ${size_y} ${size_z}"/></geometry><origin xyz="0 0 0" rpy="0 0 0"/></collision>
-      <inertial><mass value="${mass}"/><origin xyz="0 0 0" rpy="0 0 0"/><inertia ixx="0.00104" iyy="0.00229" izz="0.00271"/></inertial>
-    </link>
-  </xacro:macro>
-  <xacro:macro name="bucket_wall" params="name size_x size_y size_z mass ixx iyy izz material">
-    <link name="${name}">
-      <visual><geometry><box size="${size_x} ${size_y} ${size_z}"/></geometry><origin xyz="0 0 0" rpy="0 0 0"/><material name="${material}"/></visual>
-      <collision><geometry><box size="${size_x} ${size_y} ${size_z}"/></geometry><origin xyz="0 0 0" rpy="0 0 0"/></collision>
-      <inertial><mass value="${mass}"/><origin xyz="0 0 0" rpy="0 0 0"/><inertia ixx="${ixx}" iyy="${iyy}" izz="${izz}"/></inertial>
-    </link>
-  </xacro:macro>
-  <!-- ==================== JOINT MACROS ==================== -->
-  <xacro:macro name="bucket_joint" params="name parent child xyz rpy">
+    <!--  MATERIALS MACRO  -->
+    <xacro:macro name="define_materials">
+    <material name="grey">
+        <color rgba="0.7 0.7 0.7 1"/>
+    </material>
+    <material name="green">
+        <color rgba="0 0.6 0 1"/>
+    </material>
+    <material name="white">
+        <color rgba="1 1 1 1"/>
+    </material>
+    <!-- GAZEBO SENSOR MACROS -->
+    <!-- Lidar plugin macro -->
+    <xacro:macro name="gazebo_lidar_plugin" params="reference name update_rate samples resolution min_angle max_angle min_range max_range range_res">
+        <gazebo reference="${reference}">
+            <sensor name="${name}" type="lidar">
+                <update_rate>${update_rate}</update_rate>
+                <lidar>
+                    <horizontal>
+                        <samples>${samples}</samples>
+                        <resolution>${resolution}</resolution>
+                        <min_angle>${min_angle}</min_angle>
+                        <max_angle>${max_angle}</max_angle>
+                    </horizontal>
+                    <range>
+                        <min>${min_range}</min>
+                        <max>${max_range}</max>
+                        <resolution>${range_res}</resolution>
+                    </range>
+                </lidar>
+            </sensor>
+        </gazebo>
+    </xacro:macro>
+    <!-- Camera plugin macro -->
+    <xacro:macro name="gazebo_camera_plugin" params="reference name update_rate fov width height format near far">
+        <gazebo reference="${reference}">
+            <sensor name="${name}" type="camera">
+                <update_rate>${update_rate}</update_rate>
+                <camera>
+                    <horizontal_fov>${fov}</horizontal_fov>
+                    <image>
+                        <width>${width}</width>
+                        <height>${height}</height>
+                        <format>${format}</format>
+                    </image>
+                    <clip>
+                        <near>${near}</near>
+                        <far>${far}</far>
+                    </clip>
+                </camera>
+            </sensor>
+        </gazebo>
+    </xacro:macro>
+    <!-- IMU plugin macro -->
+    <xacro:macro name="gazebo_imu_plugin" params="reference name update_rate">
+        <gazebo reference="${reference}">
+            <sensor name="${name}" type="imu">
+                <update_rate>${update_rate}</update_rate>
+                <imu>
+                    <angular_velocity/>
+                    <linear_acceleration/>
+                </imu>
+            </sensor>
+        </gazebo>
+    </xacro:macro>
+    <!-- ==================== GAZEBO SENSOR CALLS ==================== -->
+    <!-- Lidar -->
+    <xacro:gazebo_lidar_plugin
+        reference="lidar"
+        name="lidar_sensor"
+        update_rate="30"
+        samples="720" resolution="1"
+        min_angle="-3.14" max_angle="3.14"
+        min_range="0.1" max_range="30.0"
+        range_res="0.01"/>
+    <!-- Camera -->
+    <xacro:gazebo_camera_plugin
+        reference="camera_link"
+        name="camera_sensor"
+        update_rate="30"
+        fov="1.57"
+        width="640" height="480"
+        format="R8G8B8"
+        near="0.1" far="50.0"/>
+    <!-- IMU -->
+    <xacro:gazebo_imu_plugin
+        reference="imu_link"
+        name="imu_sensor"
+        update_rate="100"/>
+    </xacro:macro>
+    <!-- MATERIALS CALL -->
+    <xacro:define_materials/>
+    <!-- DUMMY LINK AS A FRAME -->
+    <link name="base_footprint"/>
+    <link name="bucket"/>
+    <!--  LINK MACROS  -->
+    <xacro:macro name="box_link" params="name size_x size_y size_z origin_xyz origin_rpy mass material ixx:=0 iyy:=0 izz:=0 ixy:=0 ixz:=0 iyz:=0">
+        <link name="${name}">
+            <visual>
+                <geometry><box size="${size_x} ${size_y} ${size_z}"/></geometry>
+                <origin xyz="${origin_xyz}" rpy="${origin_rpy}"/>
+                <material name="${material}"/>
+            </visual>
+            <collision>
+                <geometry><box size="${size_x} ${size_y} ${size_z}"/></geometry>
+                <origin xyz="${origin_xyz}" rpy="${origin_rpy}"/>
+            </collision>
+            <inertial>
+                <mass value="${mass}"/>
+                <origin xyz="${origin_xyz}" rpy="${origin_rpy}"/>
+                <inertia ixx="${ixx}" iyy="${iyy}" izz="${izz}" ixy="${ixy}" ixz="${ixz}" iyz="${iyz}"/>
+            </inertial>
+        </link>
+    </xacro:macro>
+        <xacro:macro name="cylinder_link" params="name radius length origin_xyz origin_rpy material mass:=0.1 ixx:=0 iyy:=0 izz:=0">
+            <link name="${name}">
+                <visual>
+                    <geometry><cylinder radius="${radius}" length="${length}"/></geometry>
+                    <origin xyz="${origin_xyz}" rpy="${origin_rpy}"/>
+                    <material name="${material}"/>
+                </visual>
+                <collision>
+                    <geometry><cylinder radius="${radius}" length="${length}"/></geometry>
+                    <origin xyz="${origin_xyz}" rpy="${origin_rpy}"/>
+            </collision>
+            <inertial>
+                <mass value="${mass}"/>
+                <origin xyz="${origin_xyz}" rpy="${origin_rpy}"/>
+                <inertia ixx="${ixx}" iyy="${iyy}" izz="${izz}"/>
+            </inertial>
+            </link>
+        </xacro:macro>
+    <!-- LINK CALLS  -->
+    <!-- Base link -->
+    <xacro:box_link
+    name="base_link"
+    size_x="0.6" size_y="0.4" size_z="0.2"
+    origin_xyz="0 0 0.1" origin_rpy="0 0 0"
+    mass="10.0" material="green"
+    ixx="0.183" iyy="0.333" izz="0.500"/>
+    <!-- Lidar -->
+    <xacro:cylinder_link
+    name="lidar"
+    radius="0.1" length="0.05"
+    origin_xyz="0 0 0" origin_rpy="0 0 0"
+    material="white"/>
+    <!-- Camera -->
+    <xacro:box_link
+    name="camera_link"
+    size_x="0.02" size_y="0.07" size_z="0.02"
+    origin_xyz="0 0 0" origin_rpy="0 0 0"
+    mass="0.1" material="white"
+    ixx="0.0001" iyy="0.0001" izz="0.0001"/>
+    <!-- IMU -->
+    <xacro:box_link
+    name="imu_link"
+    size_x="0.025" size_y="0.08" size_z="0.01"
+    origin_xyz="0 0 0" origin_rpy="0 0 0"
+    mass="0.05" material="grey"
+    ixx="0.00002" iyy="0.00002" izz="0.00002"/>
+    <!--  WHEEL MACRO  -->
+    <xacro:macro name="wheel_link" params="name radius length origin_rpy mass material ixx:=0.00375 iyy:=0.00375 izz:=0.005">
+        <link name="${name}">
+            <visual>
+                <geometry>
+                    <cylinder radius="${radius}" length="${length}"/>
+                </geometry>
+                <origin xyz="0 0 0" rpy="${origin_rpy}"/>
+                <material name="${material}"/>
+            </visual>
+            <collision>
+                <geometry>
+                    <cylinder radius="${radius}" length="${length}"/>
+                </geometry>
+                <origin xyz="0 0 0" rpy="${origin_rpy}"/>
+            </collision>
+            <inertial>
+                <mass value="${mass}"/>
+                <origin xyz="0 0 0" rpy="${origin_rpy}"/>
+                <inertia ixx="${ixx}" iyy="${iyy}" izz="${izz}" ixy="0.0" ixz="0.0" iyz="0.0"/>
+            </inertial>
+        </link>
+    </xacro:macro>
+<!--  WHEEL CALLS  -->
+    <xacro:wheel_link
+        name="left_wheel"
+        radius="0.1" length="0.05"
+        origin_rpy="1.57 0 0"
+        mass="1.0"
+        material="white"/>
+    <xacro:wheel_link
+        name="right_wheel"
+        radius="0.1" length="0.05"
+        origin_rpy="1.57 0 0"
+        mass="1.0"
+        material="white"/>
+   <!--  CASTER WHEEL MACRO  -->
+    <xacro:macro name="caster_link" params="name radius mass material ixx:=0.001 iyy:=0.001 izz:=0.001">
+        <link name="${name}">
+            <visual>
+                <geometry>
+                    <sphere radius="${radius}"/>
+                </geometry>
+                <origin xyz="0 0 0" rpy="0 0 0"/>
+                <material name="${material}"/>
+            </visual>
+            <collision>
+                <geometry>
+                    <sphere radius="${radius}"/>
+                </geometry>
+                <origin xyz="0 0 0" rpy="0 0 0"/>
+            </collision>
+            <inertial>
+                <mass value="${mass}"/>
+                <origin xyz="0 0 0" rpy="0 0 0"/>
+                <inertia ixx="${ixx}" iyy="${iyy}" izz="${izz}" ixy="0.0" ixz="0.0" iyz="0.0"/>
+            </inertial>
+        </link>
+    </xacro:macro>
+    <!--  CASTER WHEEL CALL  -->
+    <xacro:caster_link
+        name="caster_wheel"
+        radius="0.05"
+        mass="0.5"
+        material="white"/>
+    <!--  WING MACRO -->
+    <xacro:macro name="wing_link" params="name size_x size_y size_z mass material ixx:=0.00104 iyy:=0.00229 izz:=0.00271">
+        <link name="${name}">
+            <visual>
+                <geometry>
+                    <box size="${size_x} ${size_y} ${size_z}"/>
+                </geometry>
+                <origin xyz="0 0 0" rpy="0 0 0"/>
+                <material name="${material}"/>
+            </visual>
+            <collision>
+                <geometry>
+                    <box size="${size_x} ${size_y} ${size_z}"/>
+                </geometry>
+                <origin xyz="0 0 0" rpy="0 0 0"/>
+            </collision>
+            <inertial>
+                <mass value="${mass}"/>
+                <origin xyz="0 0 0" rpy="0 0 0"/>
+                <inertia ixx="${ixx}" iyy="${iyy}" izz="${izz}" ixy="0.0" ixz="0.0" iyz="0.0"/>
+            </inertial>
+        </link>
+    </xacro:macro>
+    <!--  WING CALLS -->
+    <xacro:wing_link
+        name="scoop_left_wing"
+        size_x="0.1" size_y="0.040" size_z="0.05"
+        mass="0.5"
+        material="white"/>
+    <xacro:wing_link
+        name="scoop_right_wing"
+        size_x="0.1" size_y="0.040" size_z="0.05"
+        mass="0.5"
+        material="white"/>
+    <!-- BUCKET WALL CALLS  -->
+    <!-- Bottom wall -->
+    <xacro:box_link
+        name="bucket_bottom"
+        size_x="0.1" size_y="0.3" size_z="0.01"
+        origin_xyz="0 0 0" origin_rpy="0 0 0"
+        mass="0.3" material="white"
+        ixx="0.000075" iyy="0.00075" izz="0.00075"/>
+    <!-- Back wall -->
+    <xacro:box_link
+        name="bucket_back_wall"
+        size_x="0.01" size_y="0.3" size_z="0.15"
+        origin_xyz="0 0 0" origin_rpy="0 0 0"
+        mass="0.5" material="white"
+        ixx="0.0010" iyy="0.0031" izz="0.0031"/>
+    <!-- Left wall -->
+    <xacro:box_link
+        name="bucket_left_wall"
+        size_x="0.1" size_y="0.006" size_z="0.15"
+        origin_xyz="0 0 0" origin_rpy="0 0 0"
+        mass="0.2" material="white"
+        ixx="0.00038" iyy="0.00013" izz="0.00042"/>
+    <!-- Right wall -->
+    <xacro:box_link
+        name="bucket_right_wall"
+        size_x="0.1" size_y="0.006" size_z="0.15"
+        origin_xyz="0 0 0" origin_rpy="0 0 0"
+        mass="0.2" material="white"
+        ixx="0.00038" iyy="0.00013" izz="0.00042"/>
+   <!--  BUCKET FRONT LIP CALL -->
+    <xacro:box_link
+        name="bucket_front_lip"
+        size_x="0.02" size_y="0.3" size_z="0.005"
+        origin_xyz="0 0 0" origin_rpy="0 0 0"
+        mass="0.1" material="white"
+        ixx="0.000019" iyy="0.00045" izz="0.00045"/>
+    <!-- BUCKET JOINT MACRO  -->
+    <xacro:macro name="bucket_joint" params="name parent child xyz rpy">
     <joint name="${name}" type="fixed">
-      <parent link="${parent}"/>
-      <child link="${child}"/>
-      <origin xyz="${xyz}" rpy="${rpy}"/>
+        <parent link="${parent}"/>
+        <child link="${child}"/>
+        <origin xyz="${xyz}" rpy="${rpy}"/>
     </joint>
-  </xacro:macro>
-  <xacro:macro name="generic_joint" params="name type parent child xyz rpy axis:='' lower:='' upper:='' effort:='' velocity:=''">
-    <joint name="${name}" type="${type}">
-      <parent link="${parent}"/>
-      <child link="${child}"/>
-      <origin xyz="${xyz}" rpy="${rpy}"/>
-      <xacro:if value="${axis != ''}"><axis xyz="${axis}"/></xacro:if>
-      <xacro:if value="${lower != ''}"><limit lower="${lower}" upper="${upper}" effort="${effort}" velocity="${velocity}"/></xacro:if>
+    </xacro:macro>
+    <!--  BUCKET JOINT CALLS  -->
+    <!-- Bottom joint -->
+    <xacro:bucket_joint
+        name="bucket_bottom_joint"
+        parent="bucket"
+        child="bucket_bottom"
+        xyz="0.38 0 0.01"
+        rpy="0 0 0"/>
+    <!-- Back wall joint -->
+    <xacro:bucket_joint
+        name="bucket_back_wall_joint"
+        parent="bucket"
+        child="bucket_back_wall"
+        xyz="0.325 0 0.08"
+        rpy="0 0 0"/>
+    <!-- Left wall joint -->
+    <xacro:bucket_joint
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
Commit message: Fixed the lidar visual in rviz. Syntax issue fixed

File: urdf/Robot.xacro (robot description, xacro)
@@ -115,22 +115,22 @@
         </link>
     </xacro:macro>
-        <xacro:macro name="cylinder_link" params="name radius length origin_xyz origin_rpy material mass:=0.1 ixx:=0 iyy:=0 izz:=0">
-            <link name="${name}">
-                <visual>
-                    <geometry><cylinder radius="${radius}" length="${length}"/></geometry>
-                    <origin xyz="${origin_xyz}" rpy="${origin_rpy}"/>
-                    <material name="${material}"/>
-                </visual>
-                <collision>
-                    <geometry><cylinder radius="${radius}" length="${length}"/></geometry>
-                    <origin xyz="${origin_xyz}" rpy="${origin_rpy}"/>
+    <xacro:macro name="cylinder_link" params="name radius length origin_xyz origin_rpy material mass:=0.1 ixx:=0 iyy:=0 izz:=0">
+        <link name="${name}">
+            <visual>
+                <geometry><cylinder radius="${radius}" length="${length}"/></geometry>
+                <origin xyz="${origin_xyz}" rpy="${origin_rpy}"/>
+                <material name="${material}"/>
+            </visual>
+            <collision>
+                <geometry><cylinder radius="${radius}" length="${length}"/></geometry>
+                <origin xyz="${origin_xyz}" rpy="${origin_rpy}"/>
             </collision>
             <inertial>
                 <mass value="${mass}"/>
                 <origin xyz="${origin_xyz}" rpy="${origin_rpy}"/>
-                <inertia ixx="${ixx}" iyy="${iyy}" izz="${izz}"/>
+                <inertia ixx="${ixx}" iyy="${iyy}" izz="${izz}" ixy="0" ixz="0" iyz="0"/>
             </inertial>
-            </link>
-        </xacro:macro>
+        </link>
+    </xacro:macro>
     <!-- LINK CALLS  -->
     <!-- Base link -->

Commit message: Integrated ros2_control system into Robot.xacro

File: urdf/Robot.xacro (robot description, xacro)
@@ -1,4 +1,39 @@
 <?xml version="1.0"?>
 <robot xmlns:xacro="http://www.ros.org/wiki/xacro" name="autonomous_sphere_collector">
+    <ros2_control name="DiffDriveSystem" type="system">
+        <hardware>
+            <plugin>gazebo_ros2_control/GazeboSystem</plugin>
+        </hardware>
+        <!-- Left wheel joint -->
+        <joint name="base_left_wheel_joint">
+            <command_interfaces>
+                <command_interface name="velocity"/>
+            </command_interfaces>
+            <state_interfaces>
+                <state_interface name="position"/>
+                <state_interface name="velocity"/>
+            </state_interfaces>
+        </joint>
+        <!-- Right wheel joint -->
+        <joint name="base_right_wheel_joint">
+            <command_interfaces>
+                <command_interface name="velocity"/>
+            </command_interfaces>
+            <state_interfaces>
+                <state_interface name="position"/>
+                <state_interface name="velocity"/>
+            </state_interfaces>
+        </joint>
+        <!-- Left wing joint -->
+        <joint name="scoop_left_wing_joint">
+            <command_interfaces>
+                <command_interface name="position"/>
+            </command_interfaces>
+            <state_interfaces>
+                <state_interface name="position"/>
+                <state_interface name="velocity"/>
+            </state_interfaces>
+        </joint>
+    </ros2_control>
     <!--  MATERIALS MACRO  -->
     <xacro:macro name="define_materials">
