Commit message: map commited

File: urdf/autonomous_sphere_collector.urdf.xacro (robot description, xacro)
@@ -31,5 +31,5 @@
         </visual>
         <collision name="rear_caster_collision">
-            <origin xyz="-0.15 0 -0.05" rpy=" 0 0 0"/>
+            <origin xyz="-0.15 0 0" rpy=" 0 0 0"/>
             <geometry>
                 <sphere radius="0.0499"/>
@@ -37,12 +37,12 @@
         </collision>
         <visual name="rear_caster_visual">
-            <origin xyz="-0.15 0 -0.05" rpy=" 0 0 0"/>
-            <geometry>
-                <sphere radius="0.05"/>
+            <origin xyz="-0.15 0 0" rpy=" 0 0 0"/>
+            <geometry>
+                <sphere radius="0.0499"/>
             </geometry>
             <material name="blue"/>
         </visual>
         <collision name="front_caster_collision">
-            <origin xyz="0.15 0 -0.05" rpy=" 0 0 0"/>
+            <origin xyz="0.15 0 0" rpy=" 0 0 0"/>
             <geometry>
                 <sphere radius="0.0499"/>
@@ -50,7 +50,7 @@
         </collision>
         <visual name="front_caster_visual">
-            <origin xyz="0.15 0 -0.05" rpy=" 0 0 0"/>
-            <geometry>
-                <sphere radius="0.05"/>
+            <origin xyz="0.15 0 0" rpy=" 0 0 0"/>
+            <geometry>
+                <sphere radius="0.0499"/>
             </geometry>
             <material name="red"/>
@@ -58,10 +58,10 @@
     </link>
     <joint type="continuous" name="left_wheel_joint">
-        <origin xyz="0 0.225 0" rpy="0 0 0"/>
+        <origin xyz="0 0.235 -0.01" rpy="0 0 0"/>
         <child link="left_wheel"/>
         <parent link="base_link"/>
         <axis xyz="0 1 0" rpy="0 0 0"/>
-        <limit effort="100" velocity="10"/>
-        <dynamics damping="1.0" friction="1.0"/>
+        <limit effort="400" velocity="50"/>
+        <dynamics damping="0.0" friction="0.0"/>
     </joint>
         <link name="left_wheel">
@@ -86,10 +86,10 @@
         </link>
     <joint type="continuous" name="right_wheel_joint">
-        <origin xyz="0 -0.225 0" rpy="0 0 0"/>
+        <origin xyz="0 -0.235 -0.01" rpy="0 0 0"/>
         <child link="right_wheel"/>
         <parent link="base_link"/>
         <axis xyz="0 1 0" rpy="0 0 0"/>
-        <limit effort="100" velocity="10"/>
-        <dynamics damping="1.0" friction="1.0"/>
+        <limit effort="400" velocity="50"/>
+        <dynamics damping="0.0" friction="0.0"/>
     </joint>
     <link name="right_wheel">
@@ -114,6 +114,6 @@
     </link>
     <gazebo reference="left_wheel">
-        <mu1>0.2</mu1>
-        <mu2>0.2</mu2>
+        <mu1>1.0</mu1>
+        <mu2>1.0</mu2>
         <kp>1000000.0</kp>
         <kd>100.0</kd>
@@ -122,6 +122,6 @@
     </gazebo>
     <gazebo reference="right_wheel">
-        <mu1>0.2</mu1>
-        <mu2>0.2</mu2>
+        <mu1>1.0</mu1>
+        <mu2>1.0</mu2>
         <kp>1000000.0</kp>
         <kd>100.0</kd>
@@ -130,6 +130,6 @@
     </gazebo>
     <gazebo reference="base_link">
-        <mu1>0.000002</mu1>
-        <mu2>0.000002</mu2>
+        <mu1>0.0</mu1>
+        <mu2>0.0</mu2>
     </gazebo>
     <joint name="imu_joint" type="fixed">
@@ -220,17 +220,19 @@
         <joint name="left_wheel_joint">
             <command_interface name="velocity">
-                <param name="min">-10</param>
-                <param name="max">10</param>
+                <param name="min">-50</param>
+                <param name="max">50</param>
             </command_interface>
             <state_interface name="velocity"/>
             <state_interface name="position"/>
+            <state_interface name="effort"/>
         </joint>
         <joint name="right_wheel_joint">
             <command_interface name="velocity">
-                <param name="min">-10</param>
-                <param name="max">10</param>
+                <param name="min">-50</param>
+                <param name="max">50</param>
             </command_interface>
             <state_interface name="velocity"/>
             <state_interface name="position"/>
+            <state_interface name="effort"/>
         </joint>
         <joint name="scoop_pivot_joint">

Commit message: urdf and plugins modified to new settings

File: urdf/autonomous_sphere_collector.urdf.xacro (robot description, xacro)
@@ -14,9 +14,9 @@
         <inertial>
             <mass value="15.0"/>
-            <origin xyz="0.0 0 0" rpy=" 0 0 0"/>
+            <origin xyz="0.0 0 0" rpy="0 0 0"/>
             <inertia ixx="0.0625" ixy="0" ixz="0" iyy="0.2125" iyz="0" izz="0.25"/>
         </inertial>
         <collision name="collision">
-            <origin xyz="0 0 0" rpy=" 0 0 0"/>
+            <origin xyz="0 0 0" rpy="0 0 0"/>
             <geometry>
                 <box size="0.6 0.4 0.15"/>
@@ -24,5 +24,5 @@
         </collision>
         <visual name="base_link_visual">
-            <origin xyz="0 0 0" rpy=" 0 0 0"/>
+            <origin xyz="0 0 0" rpy="0 0 0"/>
             <geometry>
                 <box size="0.6 0.4 0.15"/>
@@ -30,40 +30,15 @@
             <material name="green"/>
         </visual>
-        <collision name="rear_caster_collision">
-            <origin xyz="-0.15 0 0" rpy=" 0 0 0"/>
-            <geometry>
-                <sphere radius="0.0499"/>
-            </geometry>
-        </collision>
-        <visual name="rear_caster_visual">
-            <origin xyz="-0.15 0 0" rpy=" 0 0 0"/>
-            <geometry>
-                <sphere radius="0.0499"/>
-            </geometry>
-            <material name="blue"/>
-        </visual>
-        <collision name="front_caster_collision">
-            <origin xyz="0.15 0 0" rpy=" 0 0 0"/>
-            <geometry>
-                <sphere radius="0.0499"/>
-            </geometry>
-        </collision>
-        <visual name="front_caster_visual">
-            <origin xyz="0.15 0 0" rpy=" 0 0 0"/>
-            <geometry>
-                <sphere radius="0.0499"/>
-            </geometry>
-            <material name="red"/>
-        </visual>
     </link>
-    <joint type="continuous" name="left_wheel_joint">
-        <origin xyz="0 0.235 -0.01" rpy="0 0 0"/>
-        <child link="left_wheel"/>
-        <parent link="base_link"/>
-        <axis xyz="0 1 0" rpy="0 0 0"/>
-        <limit effort="400" velocity="50"/>
-        <dynamics damping="0.0" friction="0.0"/>
-    </joint>
-        <link name="left_wheel">
+    <xacro:macro name="wheel" params="prefix x_reflect y_reflect">
+        <joint type="continuous" name="${prefix}_wheel_joint">
+            <origin xyz="${x_reflect * 0.2} ${y_reflect * 0.235} -0.01" rpy="0 0 0"/>
+            <child link="${prefix}_wheel"/>
+            <parent link="base_link"/>
+            <axis xyz="0 1 0" rpy="0 0 0"/>
+            <limit effort="400" velocity="50"/>
+            <dynamics damping="0.0" friction="0.0"/>
+        </joint>
+        <link name="${prefix}_wheel">
             <inertial>
                 <mass value="5.0"/>
@@ -75,58 +50,27 @@
                 <geometry>
                     <cylinder radius="0.1" length="0.05"/>
-            </geometry>
+                </geometry>
             </collision>
-                <visual name="left_wheel_visual">
-                    <origin xyz="0 0 0" rpy="0 1.5707 1.5707"/>
-                    <geometry>
-                        <cylinder radius="0.1" length="0.05"/>
-                    </geometry>
-                    <material name="black"/>
-                </visual>
+            <visual name="${prefix}_wheel_visual">
+                <origin xyz="0 0 0" rpy="0 1.5707 1.5707"/>
+                <geometry>
+                    <cylinder radius="0.1" length="0.05"/>
+                </geometry>
+                <material name="black"/>
+            </visual>
         </link>
-    <joint type="continuous" name="right_wheel_joint">
-        <origin xyz="0 -0.235 -0.01" rpy="0 0 0"/>
-        <child link="right_wheel"/>
-        <parent link="base_link"/>
-        <axis xyz="0 1 0" rpy="0 0 0"/>
-        <limit effort="400" velocity="50"/>
-        <dynamics damping="0.0" friction="0.0"/>
-    </joint>
-    <link name="right_wheel">
-        <inertial>
-            <mass value="5.0"/>
-            <origin xyz="0 0 0" rpy="0 1.5707 1.5707"/>
-            <inertia ixx="0.014" ixy="0" ixz="0" iyy="0.014" iyz="0" izz="0.025"/>
-        </inertial>
-        <collision>
-            <origin xyz="0 0 0" rpy="0 1.5707 1.5707"/>
-            <geometry>
-                <cylinder radius="0.1" length="0.05"/>
-            </geometry>
-        </collision>
-        <visual name="right_wheel_visual">
-            <origin xyz="0 0 0" rpy="0 1.5707 1.5707"/>
-            <geometry>
-                <cylinder radius="0.1" length="0.05"/>
-            </geometry>
-            <material name="black"/>
-        </visual>
-    </link>
-    <gazebo reference="left_wheel">
-        <mu1>1.0</mu1>
-        <mu2>1.0</mu2>
-        <kp>1000000.0</kp>
-        <kd>100.0</kd>
-        <minDepth>0.0001</minDepth>
-        <maxVel>1.0</maxVel>
-    </gazebo>
-    <gazebo reference="right_wheel">
-        <mu1>1.0</mu1>
-        <mu2>1.0</mu2>
-        <kp>1000000.0</kp>
-        <kd>100.0</kd>
-        <minDepth>0.0001</minDepth>
-        <maxVel>1.0</maxVel>
-    </gazebo>
+        <gazebo reference="${prefix}_wheel">
+            <mu1>1.0</mu1>
+            <mu2>1.0</mu2>
+            <kp>1000000.0</kp>
+            <kd>100.0</kd>
+            <minDepth>0.0001</minDepth>
+            <maxVel>1.0</maxVel>
+        </gazebo>
+    </xacro:macro>
+    <xacro:wheel prefix="front_left"   x_reflect="1"  y_reflect="1" />
+    <xacro:wheel prefix="front_right"  x_reflect="1"  y_reflect="-1" />
+    <xacro:wheel prefix="rear_left"    x_reflect="-1" y_reflect="1" />
+    <xacro:wheel prefix="rear_right"   x_reflect="-1" y_reflect="-1" />
     <gazebo reference="base_link">
         <mu1>0.0</mu1>
@@ -140,21 +84,21 @@
     <link name="imu_link">
         <inertial>
-                <mass value="1e-5"/>
-                <origin xyz="0 0 0" rpy="0 0 0"/>
-                <inertia ixx="1e-6" ixy="0" ixz="0" iyy="1e-6" iyz="0.0" izz="1e-6"/>
-            </inertial>
-            <collision name="collision">
-                <origin xyz="0 0 0" rpy="0 0 0"/>
-                <geometry>
-                    <box size="0.05 0.1 0.01"/>
-                </geometry>
-            </collision>
-            <visual name="visual">
-                <origin xyz="0 0 0" rpy="0 0 0"/>
-                <geometry>
-                    <box size="0.05 0.1 0.01"/>
-                </geometry>
-                <material name="white"/>
-            </visual>
+            <mass value="1e-5"/>
+            <origin xyz="0 0 0" rpy="0 0 0"/>
+            <inertia ixx="1e-6" ixy="0" ixz="0" iyy="1e-6" iyz="0.0" izz="1e-6"/>
+        </inertial>
+        <collision name="collision">
+            <origin xyz="0 0 0" rpy="0 0 0"/>
+            <geometry>
+                <box size="0.05 0.1 0.01"/>
+            </geometry>
+        </collision>
+        <visual name="visual">
+            <origin xyz="0 0 0" rpy="0 0 0"/>
+            <geometry>
+                <box size="0.05 0.1 0.01"/>
+            </geometry>
+            <material name="white"/>
+        </visual>
     </link>
     <joint type="fixed" name="scan_joint">
@@ -213,35 +157,3 @@
         </visual>
     </link>
-    <ros2_control name="GazeboSystem" type="system">
-        <hardware name="base_controller/BaseSystem">
-            <plugin>gz_ros2_control/GazeboSimSystem</plugin>
-            <param name="simulate_velocity">true</param>
-        </hardware>
-        <joint name="left_wheel_joint">
-            <command_interface name="velocity">
-                <param name="min">-50</param>
-                <param name="max">50</param>
-            </command_interface>
-            <state_interface name="velocity"/>
-            <state_interface name="position"/>
-            <state_interface name="effort"/>
-        </joint>
-        <joint name="right_wheel_joint">
-            <command_interface name="velocity">
-                <param name="min">-50</param>
-                <param name="max">50</param>
-            </command_interface>
-            <state_interface name="velocity"/>
-            <state_interface name="position"/>
-            <state_interface name="effort"/>
-        </joint>
-        <joint name="scoop_pivot_joint">
-            <command_interface name="position">
-                <param name="min">-1.5708</param>
-                <param name="max">0.610865</param>
-            </command_interface>
-            <state_interface name="position"/>
-            <state_interface name="velocity"/>
-        </joint>
-    </ros2_control>
 </robot>
